File: Hardware/Heartbeat Monitor.kicad_sch (KiCad schematic)
At the start: 0 parts

Commit message: Update
Parts:
- added J1: USB_C_Receptacle_USB2.0_14P, Package_DFN_QFN:Texas_RNQ0040A_WQFN-40-1EP_6x4mm_P0.4mm_EP4.7x2.7mm, symbol Connector:USB_C_Receptacle_USB2.0_14P
Connections:
- new net: J1.A1 (GND), J1.A12 (GND), J1.B1 (GND), J1.B12 (GND)
- new net: J1.A4 (VBUS), J1.A9 (VBUS), J1.B4 (VBUS), J1.B9 (VBUS)
Changed lines of the file:
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@@
 	(generator_version "10.0")
 	(paper "A4")
+	(symbol
+		(lib_id "Connector:USB_C_Receptacle_USB2.0_14P")
+		(at 29.21 38.1 0)
+		(unit 1)
+		(body_style 1)
+		(exclude_from_sim no)
+		(in_bom yes)
+		(on_board yes)
+		(in_pos_files yes)
+		(dnp no)
+		(fields_autoplaced yes)
+		(property "Reference" "J1"
+			(at 29.21 15.24 0)
+			(show_name no)
+			(do_not_autoplace no)
+			(effects
+				(font
+					(size 1.27 1.27)
+				)
+			)
+		)
+		(property "Value" "USB_C_Receptacle_USB2.0_14P"
+			(at 29.21 17.78 0)
+			(show_name no)
+			(do_not_autoplace no)
+			(effects
+				(font
+					(size 1.27 1.27)
+				)
+			)
+		)
+		(property "Footprint" "Package_DFN_QFN:Texas_RNQ0040A_WQFN-40-1EP_6x4mm_P0.4mm_EP4.7x2.7mm"
+			(at 33.02 38.1 0)
+			(hide yes)
+			(show_name no)
+			(do_not_autoplace no)
+			(effects
+				(font
+					(size 1.27 1.27)
+				)
+			)
+		)
+		(property "Datasheet" "https://www.usb.org/sites/default/files/documents/usb_type-c.zip"
+			(at 33.02 38.1 0)
+			(hide yes)
+			(show_name no)
+			(do_not_autoplace no)
+			(effects
+				(font
+					(size 1.27 1.27)
+				)
+			)
+		)
+		(property "Description" "USB 2.0-only 14P Type-C Receptacle connector"
+			(at 29.21 38.1 0)
+			(hide yes)
+			(show_name no)
+			(do_not_autoplace no)
+			(effects
+				(font
+					(size 1.27 1.27)
+				)
+			)
+		)
+		(pin "A1"
+		)
+		(pin "A6"
+		)
+		(pin "B6"
+		)
+		(pin "A7"
+		)
+		(pin "B1"
+		)
+		(pin "A4"
+		)
+		(pin "A9"
+		)
+		(pin "B12"
+		)
+		(pin "A5"
+		)
+		(pin "B4"
+		)
+		(pin "A12"
+		)
+		(pin "SH"
+		)
+		(pin "B9"
+		)
+		(pin "B5"
+		)
+		(pin "B7"
+		)
+		(instances
+			(project "Heartbeat Monitor"
+				(path "/ab4949ac-e668-4624-a147-a74f2884d9f8"
+					(reference "J1")
+					(unit 1)
+				)
+			)
+		)
+	)
 	(sheet_instances
 		(path "/"

Commit message: Update
Parts:
- removed J1: USB_C_Receptacle_USB2.0_14P, Package_DFN_QFN:Texas_RNQ0040A_WQFN-40-1EP_6x4mm_P0.4mm_EP4.7x2.7mm, symbol Connector:USB_C_Receptacle_USB2.0_14P
- added U1: ESP32_C3_Super_Mini, ESP32-C3-SuperMini:ESP32_C3_Super_Mini, symbol ESP32-C3-SuperMini:ESP32_C2_Super_Mini
Changed lines of the file:
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@@
 	(paper "A4")
 	(symbol
-		(lib_id "Connector:USB_C_Receptacle_USB2.0_14P")
-		(at 29.21 38.1 0)
+		(lib_id "ESP32-C3-SuperMini:ESP32_C2_Super_Mini")
+		(at 41.91 34.29 0)
 		(unit 1)
 		(body_style 1)
@@
 		(dnp no)
 		(fields_autoplaced yes)
-		(property "Reference" "J1"
-			(at 29.21 15.24 0)
+		(property "Reference" "U1"
+			(at 40.64 19.05 0)
 			(show_name no)
 			(do_not_autoplace no)
@@
 			)
 		)
-		(property "Value" "USB_C_Receptacle_USB2.0_14P"
-			(at 29.21 17.78 0)
+		(property "Value" "ESP32_C3_Super_Mini"
+			(at 40.64 21.59 0)
 			(show_name no)
 			(do_not_autoplace no)
@@
 			)
 		)
-		(property "Footprint" "Package_DFN_QFN:Texas_RNQ0040A_WQFN-40-1EP_6x4mm_P0.4mm_EP4.7x2.7mm"
-			(at 33.02 38.1 0)
+		(property "Footprint" "ESP32-C3-SuperMini:ESP32_C3_Super_Mini"
+			(at 41.91 69.85 0)
 			(hide yes)
 			(show_name no)
@@
 			)
 		)
-		(property "Datasheet" "https://www.usb.org/sites/default/files/documents/usb_type-c.zip"
-			(at 33.02 38.1 0)
+		(property "Datasheet" "https://microsoft.github.io/devicescript/devices/esp32/esp32c3-supermini"
+			(at 41.91 72.39 0)
 			(hide yes)
 			(show_name no)
@@
 			)
 		)
-		(property "Description" "USB 2.0-only 14P Type-C Receptacle connector"
-			(at 29.21 38.1 0)
-			(hide yes)
+		(property "Description" ""
+			(at 41.91 34.29 0)
 			(show_name no)
 			(do_not_autoplace no)
@@
 			)
 		)
-		(pin "A1"
+		(pin "5"
 		)
-		(pin "A6"
+		(pin "8"
 		)
-		(pin "B6"
+		(pin "9"
 		)
-		(pin "A7"
+		(pin "10"
 		)
-		(pin "B1"
+		(pin "20"
 		)
-		(pin "A4"
+		(pin "21"
 		)
-		(pin "A9"
+		(pin "1"
 		)
-		(pin "B12"
+		(pin "-2"
 		)
-		(pin "A5"
+		(pin "4"
 		)
-		(pin "B4"
+		(pin "0"
 		)
-		(pin "A12"
+		(pin "7"
 		)
-		(pin "SH"
+		(pin "6"
 		)
-		(pin "B9"
+		(pin "2"
 		)
-		(pin "B5"
+		(pin "3"
 		)
-		(pin "B7"
+		(pin "-3"
+		)
+		(pin "-1"
 		)
 		(instances
 			(project "Heartbeat Monitor"
 				(path "/ab4949ac-e668-4624-a147-a74f2884d9f8"
-					(reference "J1")
+					(reference "U1")
 					(unit 1)
 				)
